File: schematics/eurogen.kicad_pcb (KiCad board)
At the start: 2 copper layers, 8 parts, among them J1 AudioJack2, J2 AudioJack2_Ground_SwitchT, J2 AudioJack2_SwitchT, J3 PJ301M-12, J4 EURO_PWR_2x5, U1 ESP32-DEVKITC-32D, U2 CODECODER-WM8731SEDS_V(SSOP28), U3 MCP3208

Commit message: schematics update
Parts:
- removed the J2 at (0.00, 0.00)
- removed the J2 at (-15.2, -7.62)
- added C1: 220p, Capacitor_THT:C_Disc_D3.0mm_W1.6mm_P2.50mm, F.Cu at (35.5, 67.0)
- added C10: 10uF, Capacitor_THT:CP_Radial_D4.0mm_P1.50mm, F.Cu at (179.1, 85.7)
- added C11: 22p, Capacitor_THT:C_Disc_D3.0mm_W1.6mm_P2.50mm, F.Cu at (186.1, 68.6)
- added C12: 22p, Capacitor_THT:C_Disc_D3.0mm_W1.6mm_P2.50mm, F.Cu at (186.1, 73.7)
- added C13: 100n, Capacitor_THT:C_Disc_D4.3mm_W1.9mm_P5.00mm, F.Cu at (224.1, 73.0)
- added C14: 100n, Capacitor_THT:C_Disc_D4.3mm_W1.9mm_P5.00mm, F.Cu at (214.0, 16.5)
- added C15: 100n, Capacitor_THT:C_Disc_D4.3mm_W1.9mm_P5.00mm, F.Cu at (243.6, 73.0)
- added C16: 100n, Capacitor_THT:C_Disc_D4.3mm_W1.9mm_P5.00mm, F.Cu at (224.6, 24.0)
- added C17: 220uf, Capacitor_THT:C_Radial_D6.3mm_H5.0mm_P2.50mm, F.Cu at (32.0, 94.0)
- added C18: 220uf, Capacitor_THT:C_Radial_D6.3mm_H5.0mm_P2.50mm, F.Cu at (40.0, 94.0)
- added C19: 47uf, Capacitor_THT:C_Radial_D6.3mm_H5.0mm_P2.50mm, F.Cu at (168.6, 17.9)
- added C2: 10uF, Capacitor_THT:CP_Radial_D4.0mm_P1.50mm, F.Cu at (41.7, 67.0)
- added C20: 47uf, Capacitor_THT:C_Radial_D6.3mm_H5.0mm_P2.50mm, F.Cu at (178.0, 18.0)
- added C21: 100n, Capacitor_THT:C_Disc_D4.3mm_W1.9mm_P5.00mm, F.Cu at (170.0, 4.50)
- added C22: 47uf, Capacitor_THT:C_Radial_D6.3mm_H5.0mm_P2.50mm, F.Cu at (193.1, 18.0)
- added C23: 100n, Capacitor_THT:C_Disc_D4.3mm_W1.9mm_P5.00mm, F.Cu at (189.1, 4.50)
- added C24: 220p, Capacitor_THT:C_Disc_D3.0mm_W1.6mm_P2.50mm, F.Cu at (120.0, 85.0)
- added C25: 220p, Capacitor_THT:C_Disc_D3.0mm_W1.6mm_P2.50mm, F.Cu at (148.0, 84.5)
- added C26: 1uF, Capacitor_THT:CP_Radial_D4.0mm_P1.50mm, F.Cu at (127.7, 83.4)
- added C27: 1uF, Capacitor_THT:CP_Radial_D4.0mm_P1.50mm, F.Cu at (156.0, 83.0)
- added C3: 220p, Capacitor_THT:C_Disc_D3.0mm_W1.6mm_P2.50mm, F.Cu at (35.0, 85.0)
- added C4: 10uF, Capacitor_THT:CP_Radial_D4.0mm_P1.50mm, F.Cu at (41.7, 84.8)
- added C5: 100n, Capacitor_THT:C_Disc_D4.3mm_W1.9mm_P5.00mm, F.Cu at (179.8, 47.0)
- added C6: 10uF, Capacitor_THT:CP_Radial_D4.0mm_P1.50mm, F.Cu at (178.4, 51.4)
- added C7: 22p, Capacitor_THT:C_Disc_D3.0mm_W1.6mm_P2.50mm, F.Cu at (186.1, 34.3)
- added C8: 22p, Capacitor_THT:C_Disc_D3.0mm_W1.6mm_P2.50mm, F.Cu at (186.1, 39.4)
- added C9: 100n, Capacitor_THT:C_Disc_D4.3mm_W1.9mm_P5.00mm, F.Cu at (179.8, 81.3)
- added D1: LED, LED_THT:LED_D5.0mm, F.Cu at (15.1, 7.00)
- added D2: LED, LED_THT:LED_D5.0mm, F.Cu at (39.2, 7.00)
- added D3: LED, LED_THT:LED_D5.0mm, F.Cu at (63.8, 7.00)
- added D4: LED, LED_THT:LED_D5.0mm, F.Cu at (87.8, 7.00)
- added H1: MountingHole_Pad, MountingHole:MountingHole_3.2mm_M3_Pad, F.Cu at (103.0, 68.5)
- added H2: MountingHole_Pad, MountingHole:MountingHole_3.2mm_M3_Pad, F.Cu at (-2.62, 92.8)
- added H3: MountingHole_Pad, MountingHole:MountingHole_3.2mm_M3_Pad, F.Cu at (254.2, 93.4)
- added H4: MountingHole_Pad, MountingHole:MountingHole_3.2mm_M3_Pad, F.Cu at (-2.69, 6.05)
- added H5: MountingHole_Pad, MountingHole:MountingHole_3.2mm_M3_Pad, F.Cu at (255.2, 5.13)
- added H6: MountingHole_Pad, MountingHole:MountingHole_3.2mm_M3_Pad, F.Cu at (-2.46, 53.1)
- added H7: MountingHole_Pad, MountingHole:MountingHole_3.2mm_M3_Pad, F.Cu at (103.3, 95.5)
- added J10: cv in 2, Eurocad:PJ301M-12, F.Cu at (54.0, 85.9)
- added J11: cv in 4, Eurocad:PJ301M-12, F.Cu at (66.6, 85.9)
- added J12: cv in 3, Eurocad:PJ301M-12, F.Cu at (66.6, 68.0)
- added J13: stereo headphones out, Eurocad:PJ301M-12, F.Cu at (8.00, 84.0)
- added J2: EURO_PWR_2x5, Connector_PinHeader_2.54mm:PinHeader_2x05_P2.54mm_Vertical, F.Cu at (148.6, 5.00)
- added J5: codec out 1, Eurocad:PJ301M-12, F.Cu at (79.7, 67.9)
- added J6: codec out 2, Eurocad:PJ301M-12, F.Cu at (79.7, 85.7)
- added J7: codec out 3, Eurocad:PJ301M-12, F.Cu at (93.0, 67.9)
- added J8: codec out 4, Eurocad:PJ301M-12, F.Cu at (93.0, 85.7)
- added J9: cv in 1, Eurocad:PJ301M-12, F.Cu at (54.0, 68.0)
- added R1: 36k, Resistor_THT:R_Axial_DIN0207_L6.3mm_D2.5mm_P7.62mm_Horizontal, F.Cu at (41.0, 57.0)
- added R10: 47r, Resistor_THT:R_Axial_DIN0207_L6.3mm_D2.5mm_P7.62mm_Horizontal, F.Cu at (168.9, 68.6)
- added R11: 4k7, Resistor_THT:R_Axial_DIN0207_L6.3mm_D2.5mm_P7.62mm_Horizontal, F.Cu at (232.6, 55.0)
- added R12: 26k9, Resistor_THT:R_Axial_DIN0207_L6.3mm_D2.5mm_P7.62mm_Horizontal, F.Cu at (227.6, 68.5)
- added R13: 1k, Resistor_THT:R_Axial_DIN0207_L6.3mm_D2.5mm_P7.62mm_Horizontal, F.Cu at (210.8, 63.5)
- added R14: 2k2, Resistor_THT:R_Axial_DIN0207_L6.3mm_D2.5mm_P7.62mm_Horizontal, F.Cu at (215.5, 5.00)
- added R15: 29k5, Resistor_THT:R_Axial_DIN0207_L6.3mm_D2.5mm_P7.62mm_Horizontal, F.Cu at (232.6, 60.0)
- added R16: 29k5, Resistor_THT:R_Axial_DIN0207_L6.3mm_D2.5mm_P7.62mm_Horizontal, F.Cu at (255.6, 77.0)
- added R17: 4k7, Resistor_THT:R_Axial_DIN0207_L6.3mm_D2.5mm_P7.62mm_Horizontal, F.Cu at (250.6, 84.5)
- added R18: 26k9, Resistor_THT:R_Axial_DIN0207_L6.3mm_D2.5mm_P7.62mm_Horizontal, F.Cu at (245.6, 77.0)
- added R19: 47k, Resistor_THT:R_Axial_DIN0207_L6.3mm_D2.5mm_P7.62mm_Horizontal, F.Cu at (12.0, 96.0)
- added R2: 6k8, Resistor_THT:R_Axial_DIN0207_L6.3mm_D2.5mm_P7.62mm_Horizontal, F.Cu at (33.4, 62.0)
- added R20: 47k, Resistor_THT:R_Axial_DIN0207_L6.3mm_D2.5mm_P7.62mm_Horizontal, F.Cu at (17.0, 96.0)
- added R21: 1k, Resistor_THT:R_Axial_DIN0207_L6.3mm_D2.5mm_P7.62mm_Horizontal, F.Cu at (210.9, 74.9)
- added R22: 29k5, Resistor_THT:R_Axial_DIN0207_L6.3mm_D2.5mm_P7.62mm_Horizontal, F.Cu at (240.1, 85.5)
- added R23: 29k5, Resistor_THT:R_Axial_DIN0207_L6.3mm_D2.5mm_P7.62mm_Horizontal, F.Cu at (255.6, 60.5)
- added R24: 4k7, Resistor_THT:R_Axial_DIN0207_L6.3mm_D2.5mm_P7.62mm_Horizontal, F.Cu at (232.6, 90.5)
- added R25: 4k7, Resistor_THT:R_Axial_DIN0207_L6.3mm_D2.5mm_P7.62mm_Horizontal, F.Cu at (250.6, 60.4)
- added R26: 26k9, Resistor_THT:R_Axial_DIN0207_L6.3mm_D2.5mm_P7.62mm_Horizontal, F.Cu at (227.6, 84.5)
- added R27: 26k9, Resistor_THT:R_Axial_DIN0207_L6.3mm_D2.5mm_P7.62mm_Horizontal, F.Cu at (245.6, 68.0)
- added R28: 1k, Resistor_THT:R_Axial_DIN0207_L6.3mm_D2.5mm_P7.62mm_Horizontal, F.Cu at (210.9, 80.6)
- added R29: 1k, Resistor_THT:R_Axial_DIN0207_L6.3mm_D2.5mm_P7.62mm_Horizontal, F.Cu at (210.8, 69.2)
- added R3: 36k, Resistor_THT:R_Axial_DIN0207_L6.3mm_D2.5mm_P7.62mm_Horizontal, F.Cu at (41.1, 75.1)
- added R30: 200k, Resistor_THT:R_Axial_DIN0207_L6.3mm_D2.5mm_P7.62mm_Horizontal, F.Cu at (240.6, 11.5)
- added R31: 100k, Resistor_THT:R_Axial_DIN0207_L6.3mm_D2.5mm_P7.62mm_Horizontal, F.Cu at (233.1, 7.54)
- added R32: 33k, Resistor_THT:R_Axial_DIN0207_L6.3mm_D2.5mm_P7.62mm_Horizontal, F.Cu at (227.6, 19.5)
- added R33: 200k, Resistor_THT:R_Axial_DIN0207_L6.3mm_D2.5mm_P7.62mm_Horizontal, F.Cu at (240.1, 37.0)
- added R34: 100k, Resistor_THT:R_Axial_DIN0207_L6.3mm_D2.5mm_P7.62mm_Horizontal, F.Cu at (240.1, 42.0)
- added R35: 33k, Resistor_THT:R_Axial_DIN0207_L6.3mm_D2.5mm_P7.62mm_Horizontal, F.Cu at (227.6, 27.0)
- added R36: 200k, Resistor_THT:R_Axial_DIN0207_L6.3mm_D2.5mm_P7.62mm_Horizontal, F.Cu at (250.6, 20.5)
- added R37: 200k, Resistor_THT:R_Axial_DIN0207_L6.3mm_D2.5mm_P7.62mm_Horizontal, F.Cu at (250.6, 25.5)
- added R38: 100k, Resistor_THT:R_Axial_DIN0207_L6.3mm_D2.5mm_P7.62mm_Horizontal, F.Cu at (255.6, 20.5)
- added R39: 100k, Resistor_THT:R_Axial_DIN0207_L6.3mm_D2.5mm_P7.62mm_Horizontal, F.Cu at (255.6, 33.2)
- added R4: 6k8, Resistor_THT:R_Axial_DIN0207_L6.3mm_D2.5mm_P7.62mm_Horizontal, F.Cu at (33.4, 80.0)
- added R40: 33k, Resistor_THT:R_Axial_DIN0207_L6.3mm_D2.5mm_P7.62mm_Horizontal, F.Cu at (245.6, 21.2)
- added R41: 33k, Resistor_THT:R_Axial_DIN0207_L6.3mm_D2.5mm_P7.62mm_Horizontal, F.Cu at (245.6, 25.9)
- added R42: 4r7, Resistor_THT:R_Axial_DIN0207_L6.3mm_D2.5mm_P7.62mm_Horizontal, F.Cu at (164.5, 12.0)
- added R43: 10k, Resistor_THT:R_Axial_DIN0207_L6.3mm_D2.5mm_P7.62mm_Horizontal, F.Cu at (27.0, 47.0)
- added R44: 10k, Resistor_THT:R_Axial_DIN0207_L6.3mm_D2.5mm_P7.62mm_Horizontal, F.Cu at (60.0, 54.0)
- added R45: 5k6, Resistor_THT:R_Axial_DIN0207_L6.3mm_D2.5mm_P7.62mm_Horizontal, F.Cu at (107.0, 81.0)
- added R46: 5k6, Resistor_THT:R_Axial_DIN0207_L6.3mm_D2.5mm_P7.62mm_Horizontal, F.Cu at (135.0, 81.0)
- added R47: 5k6, Resistor_THT:R_Axial_DIN0207_L6.3mm_D2.5mm_P7.62mm_Horizontal, F.Cu at (107.0, 86.0)
- added R48: 5k6, Resistor_THT:R_Axial_DIN0207_L6.3mm_D2.5mm_P7.62mm_Horizontal, F.Cu at (135.0, 86.0)
- added R49: 220r, Resistor_THT:R_Axial_DIN0207_L6.3mm_D2.5mm_P7.62mm_Horizontal, F.Cu at (25.1, 3.38)
- added R5: 470r, Resistor_THT:R_Axial_DIN0207_L6.3mm_D2.5mm_P7.62mm_Horizontal, F.Cu at (112.1, 61.0)
- added R50: 220r, Resistor_THT:R_Axial_DIN0207_L6.3mm_D2.5mm_P7.62mm_Horizontal, F.Cu at (49.5, 3.17)
- added R51: 220r, Resistor_THT:R_Axial_DIN0207_L6.3mm_D2.5mm_P7.62mm_Horizontal, F.Cu at (73.7, 3.81)
- added R52: 220r, Resistor_THT:R_Axial_DIN0207_L6.3mm_D2.5mm_P7.62mm_Horizontal, F.Cu at (97.2, 3.81)
- added R53: 10k, Resistor_THT:R_Axial_DIN0207_L6.3mm_D2.5mm_P7.62mm_Horizontal, F.Cu at (11.0, 54.0)
- added R54: 10k, Resistor_THT:R_Axial_DIN0207_L6.3mm_D2.5mm_P7.62mm_Horizontal, F.Cu at (86.0, 54.0)
- added R6: 470r, Resistor_THT:R_Axial_DIN0207_L6.3mm_D2.5mm_P7.62mm_Horizontal, F.Cu at (112.1, 66.5)
- added R7: 0r, Resistor_THT:R_Axial_DIN0207_L6.3mm_D2.5mm_P7.62mm_Horizontal, F.Cu at (132.6, 61.0)
- added R8: 0r, Resistor_THT:R_Axial_DIN0207_L6.3mm_D2.5mm_P7.62mm_Horizontal, F.Cu at (132.6, 66.5)
- added R9: 47r, Resistor_THT:R_Axial_DIN0207_L6.3mm_D2.5mm_P7.62mm_Horizontal, F.Cu at (170.2, 34.3)
- added RV1: R_POT, Potentiometer_THT:Potentiometer_Alps_RK09K_Single_Vertical, F.Cu at (18.0, 31.0)
- added RV2: R_POT, Potentiometer_THT:Potentiometer_Alps_RK09K_Single_Vertical, F.Cu at (43.0, 31.0)
- added RV3: R_POT, Potentiometer_THT:Potentiometer_Alps_RK09K_Single_Vertical, F.Cu at (67.0, 31.0)
- added RV4: R_POT, Potentiometer_THT:Potentiometer_Alps_RK09K_Single_Vertical, F.Cu at (92.0, 31.0)
- added SW1: SW_Push, Button_Switch_THT:SW_PUSH-12mm, F.Cu at (8.00, 41.0)
- added SW2: SW_Push, Button_Switch_THT:SW_PUSH-12mm, F.Cu at (33.0, 41.0)
- added SW3: SW_Push, Button_Switch_THT:SW_PUSH-12mm, F.Cu at (57.0, 41.0)
- added SW4: SW_Push, Button_Switch_THT:SW_PUSH-12mm, F.Cu at (83.0, 41.0)
- added U10: LM1117-3.3, Package_TO_SOT_THT:TO-92, F.Cu at (190.6, 11.0)
- added U4: WM8731-2, CODECODER-WM8731SEDS_V_SSOP28_:SSOP28-0.65-10.2X5.2MM, F.Cu at (173.0, 77.0)
- added U5: TL074, Package_DIP:DIP-14_W7.62mm_Socket, F.Cu at (232.6, 65.5)
- added U6: LM4040LP-10, Package_TO_SOT_THT:TO-92_Inline, F.Cu at (210.5, 11.5)
- added U8: MCP6004, Package_DIP:DIP-14_W7.62mm_Socket, F.Cu at (232.6, 16.5)
- added U9: LM1117-3.3, Package_TO_SOT_THT:TO-92, F.Cu at (171.0, 11.0)
- added Y1: 12.288Mhz, ECS-17:XTAL_ECS-160-20-4X, F.Cu at (181.5, 39.0)
- added Y2: 12.288Mhz, ECS-17:XTAL_ECS-160-20-4X, F.Cu at (181.2, 73.0)
- J1: value AudioJack2 -> mono line in right; footprint Connector_Audio:Jack_3.5mm_QingPu_WQP-PJ398SM_Vertical_CircularHoles -> Eurocad:PJ301M-12
- J3: value PJ301M-12 -> mono line in left
- J4: value EURO_PWR_2x5 -> stereo line in; footprint Connector_PinHeader_2.54mm:PinHeader_2x05_P2.54mm_Vertical -> Eurocad:PJ301M-12
- U2: value CODECODER-WM8731SEDS_V(SSOP28) -> WM8731-1
- U3: footprint Package_SO:SOIC-16_4.55x10.3mm_P1.27mm -> Package_DIP:DIP-16_W7.62mm_Socket
- moved J1 164.9 mm to (20.0, 84.0)
- moved J3 81.3 mm to (20.0, 68.0)
- moved U1 61.2 mm to (122.1, 28.0), turned to 180 degrees
- moved J4 54.3 mm to (8.00, 68.0)
- moved U3 54.3 mm to (148.6, 27.9)
- moved U2 25.4 mm to (173.0, 43.0), turned to 270 degrees
Connections:
- J3 pad 3: Net-(J3-Pad3) -> GND
- J4 pad 3: Net-(J4-Pad3) -> GND
- U1 pad 10: Net-(U1-Pad10) -> /button1
- U1 pad 11: Net-(U1-Pad11) -> /button3
- U1 pad 12: Net-(U1-Pad12) -> /led4
- U1 pad 13: Net-(U1-Pad13) -> /button4
- U1 pad 15: Net-(U1-Pad15) -> /button2
- U1 pad 21: Net-(U1-Pad21) -> /adc_mosi
- U1 pad 27: Net-(U1-Pad27) -> /adc_miso
- U1 pad 28: Net-(U1-Pad28) -> /adc_clk
- U1 pad 29: Net-(U1-Pad29) -> /led3
- U1 pad 3: Net-(U1-Pad3) -> /c1_bck
- U1 pad 32: Net-(U1-Pad32) -> /c2_dac
- U1 pad 33: Net-(U1-Pad33) -> /led1
- U1 pad 34: Net-(U1-Pad34) -> /led2
- U1 pad 35: Net-(U1-Pad35) -> /adc_cs
- U1 pad 4: Net-(U1-Pad4) -> /c2_lrclk
- U1 pad 5: Net-(U1-Pad5) -> /c1_lrclk
- U1 pad 6: Net-(U1-Pad6) -> /c2_bck
- U1 pad 7: Net-(U1-Pad7) -> /c2_adc
- U1 pad 8: Net-(U1-Pad8) -> /c1_adc
- U1 pad 9: Net-(U1-Pad9) -> /c1_dac
- U2 pad 1: Net-(U2-Pad1) -> +3V3
- U2 pad 10: Net-(U2-Pad10) -> /c1_rhpout
- U2 pad 11: Net-(U2-Pad11) -> GND
- U2 pad 12: Net-(U2-Pad12) -> /c1_lout
- U2 pad 13: Net-(U2-Pad13) -> /c1_rout
- U2 pad 14: Net-(U2-Pad14) -> +3.3VA
- U2 pad 15: Net-(U2-Pad15) -> GND
- U2 pad 19: Net-(U2-Pad19) -> /audio_in2
- U2 pad 20: Net-(U2-Pad20) -> /audio_in1
- U2 pad 21: Net-(U2-Pad21) -> GND
- U2 pad 22: Net-(U2-Pad22) -> GND
- U2 pad 23: Net-(U2-Pad23) -> /i2c_data
- U2 pad 24: Net-(U2-Pad24) -> /i2c_clk
- U2 pad 27: Net-(U2-Pad27) -> +3V3
- U2 pad 28: Net-(U2-Pad28) -> GND
- U2 pad 4: Net-(U2-Pad4) -> /c1_dac
- U2 pad 5: Net-(U2-Pad5) -> /c1_lrclk
- U2 pad 6: Net-(U2-Pad6) -> /c1_adc
- U2 pad 7: Net-(U2-Pad7) -> /c1_lrclk
- U2 pad 8: Net-(U2-Pad8) -> +3.3VA
- U2 pad 9: Net-(U2-Pad9) -> /c1_lhpout
- U3 pad 1: Net-(U3-Pad1) -> /adc_ch0
- U3 pad 10: Net-(U3-Pad10) -> /adc_cs
- U3 pad 11: Net-(U3-Pad11) -> /adc_mosi
- U3 pad 12: Net-(U3-Pad12) -> /adc_miso
- U3 pad 13: Net-(U3-Pad13) -> /adc_clk
- U3 pad 14: Net-(U3-Pad14) -> GND
- U3 pad 15: Net-(U3-Pad15) -> +3V3
- U3 pad 16: Net-(U3-Pad16) -> +3V3
- U3 pad 2: Net-(U3-Pad2) -> /adc_ch1
- U3 pad 3: Net-(U3-Pad3) -> /adc_ch2
- U3 pad 4: Net-(U3-Pad4) -> /adc_ch3
- U3 pad 5: Net-(U3-Pad5) -> /adc_ch4
- U3 pad 6: Net-(U3-Pad6) -> /adc_ch5
- U3 pad 7: Net-(U3-Pad7) -> /adc_ch6
- U3 pad 8: Net-(U3-Pad8) -> /adc_ch7
- U3 pad 9: Net-(U3-Pad9) -> GND
Routing:
- net +3V3: track 0.00 -> 449.3 mm, vias 0 -> 1
- net Net-(J11-Pad1): track 0.00 -> 228.0 mm
- net Net-(J9-Pad1): track 0.00 -> 212.9 mm, vias 0 -> 1
- net Net-(J12-Pad1): track 0.00 -> 207.3 mm
- net Net-(J10-Pad1): track 0.00 -> 206.9 mm, vias 0 -> 1
- net /button3: track 0.00 -> 159.9 mm
- net /c1_lhpout: track 0.00 -> 158.1 mm, vias 0 -> 1
- net /aref_-10v: track 0.00 -> 155.9 mm
- net -12V: track 0.00 -> 154.1 mm
- net /audio_in2: track 0.00 -> 151.5 mm, vias 0 -> 1
- net /c1_rhpout: track 0.00 -> 150.8 mm, vias 0 -> 1
- net /audio_in1: track 0.00 -> 149.4 mm
- net Net-(J4-Pad2): track 0.00 -> 138.6 mm
- net /adc_ch4: track 0.00 -> 138.0 mm
- net /button1: track 0.00 -> 131.3 mm
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- added copper zone on B.Cu, net GND
- added copper zone on F.Cu, net GND
Other:
- board outline added: 270 x 100 mm
- board text added: "+12V"
- board text added: "MCP3208"
- board text added: "MCP6004"
- board text added: "TL074"
- board text added: "sinneb musical instruments"
- board text added: "team i2c"
