File: schematics/eurogen.sch (KiCad schematic (older format))
At the start: 117 parts, among them J1 PJ301M-12, J10 PJ301M-12, J11 PJ301M-12, J12 PJ301M-12, J13 PJ301M-12, J14 PJ301M-12, J2 EURO_PWR_2x5, J3 PJ301M-12, J4 AudioJack3, J5 PJ301M-12, J6 PJ301M-12, J7 PJ301M-12, J8 PJ301M-12, J9 PJ301M-12, SW1 SW_Push, SW2 SW_Push, SW3 SW_Push, U1 ESP32-DEVKITC-32D, U10 LM1117-3.3, U2 CODECODER-WM8731SEDS_V(SSOP28), U3 MCP3208, U4 CODECODER-WM8731SEDS_V(SSOP28), U5 TL074, U6 LM4040LP-10, U7 MCP6004, U8 MCP6004, U9 LM1117-3.3, Y1 12.288Mhz, Y2 12.288Mhz

Commit message: schematics update
Parts:
- R22: value 28k -> 29k5
- R26: value 25k7 -> 26k9
Connections:
- net button2: now also U1.15 (IO13); no longer U1.13 (IO12)
- net c1_adc: now also U1.8 (IO33); no longer U1.7 (IO32)
- net c2_adc: no longer U1.8 (IO33)
Changed lines of the file:
@@
 P 8150 7650
 F 0 "R26" V 8357 7650 50  0000 C CNN
-F 1 "25k7" V 8266 7650 50  0000 C CNN
+F 1 "26k9" V 8266 7650 50  0000 C CNN
 F 2 "" V 8080 7650 50  0001 C CNN
 F 3 "~" H 8150 7650 50  0001 C CNN
@@
 P 7400 7400
 F 0 "R22" V 7607 7400 50  0000 C CNN
-F 1 "28k" V 7516 7400 50  0000 C CNN
+F 1 "29k5" V 7516 7400 50  0000 C CNN
 F 2 "" V 7330 7400 50  0001 C CNN
 F 3 "~" H 7400 7400 50  0001 C CNN
@@
 Wire Wire Line
 	6050 4850 6450 4850
-Text Label 7700 1950 2    50   ~ 0
+Text Label 7700 2050 2    50   ~ 0
 c1_adc
 Text Label 11350 5000 2    50   ~ 0
@@
 Wire Wire Line
 	11350 4900 11750 4900
-Text Label 7700 2050 2    50   ~ 0
-c2_adc
 Wire Wire Line
 	7700 2050 7950 2050
@@
 Text Label 7700 2250 2    50   ~ 0
 button1
-Text Label 7700 2550 2    50   ~ 0
+Text Label 7700 2750 2    50   ~ 0
 button2
 Text Label 12050 1600 2    50   ~ 0

Commit message: schematics update
Parts:
- removed J14, J3: PJ301M-12, Eurocad:PJ301M-12, symbol eurogen-rescue:PJ301M-12-eurocad
- removed J4: AudioJack3, symbol Connector:AudioJack3
- removed U7: MCP6004, symbol Amplifier_Operational:MCP6004
- added H1, H2, H3, H4, H5, H6, H7: MountingHole_Pad, MountingHole:MountingHole_3.2mm_M3_Pad, symbol Mechanical:MountingHole_Pad
- added J3: mono line in left, Eurocad:PJ301M-12, symbol eurocad:PJ301M-12
- added J4: stereo line in, Eurocad:PJ301M-12, symbol eurogen-rescue:PJ301M-12-eurocad
- added R54: 10k, Resistor_THT:R_Axial_DIN0207_L6.3mm_D2.5mm_P7.62mm_Horizontal, symbol Device:R
- added SW4: SW_Push, Button_Switch_THT:SW_PUSH-12mm, symbol Switch:SW_Push
- added unit 1 of U8
- added unit 5 of U8
- C1, C11, C12, C24, C25, C3, C7, C8: footprint (none) -> Capacitor_THT:C_Disc_D3.0mm_W1.6mm_P2.50mm
- C10, C2, C4, C6: footprint (none) -> Capacitor_THT:CP_Radial_D4.0mm_P1.50mm
- C13, C14, C15, C16, C21, C23, C5, C9: footprint (none) -> Capacitor_THT:C_Disc_D4.3mm_W1.9mm_P5.00mm
- C17, C18, C19, C20, C22: footprint (none) -> Capacitor_THT:C_Radial_D6.3mm_H5.0mm_P2.50mm
- C26, C27: value 10uF -> 1uF; footprint (none) -> Capacitor_THT:CP_Radial_D4.0mm_P1.50mm
- D1, D2, D3, D4: footprint (none) -> LED_THT:LED_D5.0mm
- J1: value PJ301M-12 -> mono line in right
- J10: value PJ301M-12 -> cv in 2
- J11: value PJ301M-12 -> cv in 4
- J12: value PJ301M-12 -> cv in 3
- J13: value PJ301M-12 -> stereo headphones out
- J2: footprint (none) -> Connector_PinHeader_2.54mm:PinHeader_2x05_P2.54mm_Vertical
- J5: value PJ301M-12 -> codec out 1
- J6: value PJ301M-12 -> codec out 2
- J7: value PJ301M-12 -> codec out 3
- J8: value PJ301M-12 -> codec out 4
- J9: value PJ301M-12 -> cv in 1
- R1, R10, R11, R13, R14, R17, R19, R2, R20, R21, R22, R24, R25, R26, R28, R29, R3, R30, R31, R32, R33, R34, R35, R36, R37, R38, R39, R4, R40, R41, R42, R43, R44, R49, R5, R50, R51, R52, R53, R6, R7, R8, R9: footprint (none) -> Resistor_THT:R_Axial_DIN0207_L6.3mm_D2.5mm_P7.62mm_Horizontal
- R12, R18, R27: value 27k -> 26k9; footprint (none) -> Resistor_THT:R_Axial_DIN0207_L6.3mm_D2.5mm_P7.62mm_Horizontal
- R15, R16, R23: value 27k -> 29k5; footprint (none) -> Resistor_THT:R_Axial_DIN0207_L6.3mm_D2.5mm_P7.62mm_Horizontal
- R45, R46: value 36k -> 5k6; footprint (none) -> Resistor_THT:R_Axial_DIN0207_L6.3mm_D2.5mm_P7.62mm_Horizontal
- R47, R48: value 6k8 -> 5k6; footprint (none) -> Resistor_THT:R_Axial_DIN0207_L6.3mm_D2.5mm_P7.62mm_Horizontal
- RV1, RV2, RV3, RV4: footprint (none) -> Potentiometer_THT:Potentiometer_Alps_RK09K_Single_Vertical
- SW1, SW2, SW3: footprint (none) -> Button_Switch_THT:SW_PUSH-12mm
- U10, U9: footprint (none) -> Package_TO_SOT_THT:TO-92
- U2: value CODECODER-WM8731SEDS_V(SSOP28) -> WM8731-1
- U3: footprint Package_SO:SOIC-16_4.55x10.3mm_P1.27mm -> Package_DIP:DIP-16_W7.62mm_Socket
- U4: value CODECODER-WM8731SEDS_V(SSOP28) -> WM8731-2
- U5, U8: footprint (none) -> Package_DIP:DIP-14_W7.62mm_Socket
- Y1, Y2: footprint (none) -> ECS-17:XTAL_ECS-160-20-4X
Connections:
- net +3V3: now also SW4.2, U8.4 (V+)
- net GND: now also H1.1, H2.1, H3.1, H4.1, H5.1, H6.1, H7.1, J3.3, J4.3, R54.1, U8.11 (V-), U8.3 (+)
- net adc_ch0: now also U8.1
- net c2_adc: now also U1.7 (IO32)
- net button4: now reaches U1.13 (IO12)
- net button4: now also R54.2, SW4.1
- net at R1.2: now also J3.1
- net at C18.2, R20.2: now also J13.2
- net at C17.2, R19.2: now also J13.1
- net at R30.2, R31.2, R32.1: now also U8.2 (-)
- net at R45.2: now also J4.1; no longer J13.1
- net at R46.2: now also J4.2
Other:
- note added: "regular audio line in, stereo mini-jack"
