File: kicad/eurorack_engine/power.sch (KiCad schematic (older format))
At the start: 14 parts, among them J1 EURO_PWR_2x5, U2 LM1117-3.3, U4 TL074, U5 LM4040LP-10, U6 MCP6004

Commit message: schematic update
Parts:
- added SW5: DIP_USBpwr, Button_Switch_THT:SW_DIP_SPSTx01_Slide_9.78x4.72mm_W7.62mm_P2.54mm, symbol Switch:SW_DIP_x01
- J1: symbol eurogen-rescue:EURO_PWR_2x5-eurocad -> eurorack_engine-rescue:EURO_PWR_2x5-eurocad-eurogen-rescue
Connections:
- wire segments 69 -> 70
Changed lines of the file:
@@
 $EndDescr
 $Comp
-L eurogen-rescue:EURO_PWR_2x5-eurocad J?
+L eurorack_engine-rescue:EURO_PWR_2x5-eurocad-eurogen-rescue J?
 U 1 1 5F9D8E2B
 P 5400 1700
@@
 L power:+3V3 #PWR?
 U 1 1 5F9D8E9F
-P 5350 3750
+P 5350 3050
 AR Path="/5F9D8E9F" Ref="#PWR?"  Part="1"
 AR Path="/5F9CA337/5F9D8E9F" Ref="#PWR09"  Part="1"
-F 0 "#PWR09" H 5350 3600 50  0001 C CNN
-F 1 "+3V3" H 5365 3923 50  0000 C CNN
-F 2 "" H 5350 3750 50  0001 C CNN
-F 3 "" H 5350 3750 50  0001 C CNN
-	1    5350 3750
+F 0 "#PWR09" H 5350 2900 50  0001 C CNN
+F 1 "+3V3" H 5365 3223 50  0000 C CNN
+F 2 "" H 5350 3050 50  0001 C CNN
+F 3 "" H 5350 3050 50  0001 C CNN
+	1    5350 3050
 	1    0    0    -1
 $EndComp
@@
 $EndComp
 Connection ~ 10050 1400
+$Comp
+L Switch:SW_DIP_x01 SW5
+U 1 1 5F92448C
+P 5350 3450
+F 0 "SW5" V 5304 3580 50  0000 L CNN
+F 1 "DIP_USBpwr" V 5395 3580 50  0000 L CNN
+F 2 "Button_Switch_THT:SW_DIP_SPSTx01_Slide_9.78x4.72mm_W7.62mm_P2.54mm" H 5350 3450 50  0001 C CNN
+F 3 "~" H 5350 3450 50  0001 C CNN
+	1    5350 3450
+	0    1    1    0
+$EndComp
+Wire Wire Line
+	5350 3050 5350 3150
 $EndSCHEMATC
