File: kicad/eurorack_engine/power.sch (KiCad schematic (older format))
At the start: 15 parts, among them J1 EURO_PWR_2x5, SW5 DIP_USBpwr, U2 LM1117-3.3, U4 TL074, U5 LM4040LP-10, U6 MCP6004

Commit message: updated schematics
Parts:
- removed C1, C2: 47uf, Capacitor_THT:C_Radial_D6.3mm_H5.0mm_P2.50mm, symbol Device:CP
- removed C3, C6, C7, C9: 100n, Capacitor_THT:C_Disc_D4.3mm_W1.9mm_P5.00mm, symbol Device:C
- removed C8: 100n, Capacitor_THT:C_Disc_D4.3mm_W1.9mm_P5.00mm, symbol Device:CP
- removed J1: EURO_PWR_2x5, Connector_PinHeader_2.54mm:PinHeader_2x05_P2.54mm_Vertical, symbol eurorack_engine-rescue:EURO_PWR_2x5-eurocad-eurogen-rescue
- removed R5: 4r7, Resistor_THT:R_Axial_DIN0207_L6.3mm_D2.5mm_P7.62mm_Horizontal, symbol Device:R
- removed R6: 2k2, Resistor_THT:R_Axial_DIN0207_L6.3mm_D2.5mm_P7.62mm_Horizontal, symbol Device:R
- removed SW5: DIP_USBpwr, Button_Switch_THT:SW_DIP_SPSTx01_Slide_9.78x4.72mm_W7.62mm_P2.54mm, symbol Switch:SW_DIP_x01
- removed U2: LM1117-3.3, Package_TO_SOT_THT:TO-220-3_Vertical, symbol Regulator_Linear:LM1117-3.3
- removed U4: TL074, Package_DIP:DIP-14_W7.62mm_Socket, symbol Amplifier_Operational:TL074
- removed U5: LM4040LP-10, Package_TO_SOT_THT:TO-92_Inline, symbol Reference_Voltage:LM4040LP-10
- removed U6: MCP6004, Package_DIP:DIP-14_W7.62mm_Socket, symbol Amplifier_Operational:MCP6004
