File: kicad/eurorack_engine/adc.sch (KiCad schematic (older format))
At the start: 5 parts, among them U7 MCP3208

Commit message: updated schematics
Parts:
- removed RV1, RV2, RV3, RV4: R_POT, Potentiometer_THT:Potentiometer_Alps_RK09K_Single_Vertical, symbol Device:R_POT
- removed U7: MCP3208, Package_DIP:DIP-16_W7.62mm_Socket, symbol Analog_ADC:MCP3208
