File: kicad/eurorack_engine/inout.sch (KiCad schematic (older format))
At the start: 38 parts, among them J2 cv in 2, J3 cv in 1, J4 codec out 1, J5 codec out 3, J6 cv in 4, J7 cv in 3, J8 codec out 2, J9 codec out 4, U4 TL074, U6 MCP6004

Commit message: schematic update
Parts:
- J2, J3, J4, J5, J6, J7, J8, J9: symbol eurogen-rescue:PJ301M-12-eurocad -> eurorack_engine-rescue:PJ301M-12-eurocad-eurogen-rescue
Changed lines of the file:
@@
 $EndDescr
 $Comp
-L eurogen-rescue:PJ301M-12-eurocad J?
+L eurorack_engine-rescue:PJ301M-12-eurocad-eurogen-rescue J?
 U 1 1 5FA4CC8A
 P 3700 1800
 AR Path="/5F91B719/5FA4CC8A" Ref="J?"  Part="1"
 AR Path="/5FA42CB5/5FA4CC8A" Ref="J3"  Part="1"
+AR Path="/5FA4CC8A" Ref="J3"  Part="1"
 F 0 "J3" H 3708 2175 50  0000 C CNN
 F 1 "cv in 1" H 3708 2084 50  0000 C CNN
@@
 CV in -> 0/3V3\n
 $Comp
-L eurogen-rescue:PJ301M-12-eurocad J?
+L eurorack_engine-rescue:PJ301M-12-eurocad-eurogen-rescue J?
 U 1 1 5FA4CCBC
 P 3650 3600
 AR Path="/5F91B719/5FA4CCBC" Ref="J?"  Part="1"
 AR Path="/5FA42CB5/5FA4CCBC" Ref="J2"  Part="1"
+AR Path="/5FA4CCBC" Ref="J2"  Part="1"
 F 0 "J2" H 3658 3975 50  0000 C CNN
 F 1 "cv in 2" H 3658 3884 50  0000 C CNN
@@
 CV in -> 0/3V3\n
 $Comp
-L eurogen-rescue:PJ301M-12-eurocad J?
+L eurorack_engine-rescue:PJ301M-12-eurocad-eurogen-rescue J?
 U 1 1 5FA4CCEE
 P 8250 1800
 AR Path="/5F91B719/5FA4CCEE" Ref="J?"  Part="1"
 AR Path="/5FA42CB5/5FA4CCEE" Ref="J7"  Part="1"
+AR Path="/5FA4CCEE" Ref="J7"  Part="1"
 F 0 "J7" H 8258 2175 50  0000 C CNN
 F 1 "cv in 3" H 8258 2084 50  0000 C CNN
@@
 CV in -> 0/3V3\n
 $Comp
-L eurogen-rescue:PJ301M-12-eurocad J?
+L eurorack_engine-rescue:PJ301M-12-eurocad-eurogen-rescue J?
 U 1 1 5FA4CD20
 P 8200 3600
 AR Path="/5F91B719/5FA4CD20" Ref="J?"  Part="1"
 AR Path="/5FA42CB5/5FA4CD20" Ref="J6"  Part="1"
+AR Path="/5FA4CD20" Ref="J6"  Part="1"
 F 0 "J6" H 8208 3975 50  0000 C CNN
 F 1 "cv in 4" H 8208 3884 50  0000 C CNN
@@
 CODEC out -> -5/+5V
 $Comp
-L eurogen-rescue:PJ301M-12-eurocad J?
+L eurorack_engine-rescue:PJ301M-12-eurocad-eurogen-rescue J?
 U 1 1 5FA6A3E2
 P 5900 5700
 AR Path="/5F91B719/5FA6A3E2" Ref="J?"  Part="1"
 AR Path="/5FA42CB5/5FA6A3E2" Ref="J4"  Part="1"
+AR Path="/5FA6A3E2" Ref="J4"  Part="1"
 F 0 "J4" H 5908 6075 50  0000 C CNN
 F 1 "codec out 1" H 5908 5984 50  0000 C CNN
@@
 CODEC out -> -5/+5V
 $Comp
-L eurogen-rescue:PJ301M-12-eurocad J?
+L eurorack_engine-rescue:PJ301M-12-eurocad-eurogen-rescue J?
 U 1 1 5FB577EA
 P 5900 7400
 AR Path="/5F91B719/5FB577EA" Ref="J?"  Part="1"
 AR Path="/5FA42CB5/5FB577EA" Ref="J5"  Part="1"
+AR Path="/5FB577EA" Ref="J5"  Part="1"
 F 0 "J5" H 5908 7775 50  0000 C CNN
 F 1 "codec out 3" H 5908 7684 50  0000 C CNN
@@
 CODEC out -> -5/+5V
 $Comp
-L eurogen-rescue:PJ301M-12-eurocad J?
+L eurorack_engine-rescue:PJ301M-12-eurocad-eurogen-rescue J?
 U 1 1 5FB7B8C3
 P 10950 5700
 AR Path="/5F91B719/5FB7B8C3" Ref="J?"  Part="1"
 AR Path="/5FA42CB5/5FB7B8C3" Ref="J8"  Part="1"
+AR Path="/5FB7B8C3" Ref="J8"  Part="1"
 F 0 "J8" H 10958 6075 50  0000 C CNN
 F 1 "codec out 2" H 10958 5984 50  0000 C CNN
@@
 CODEC out -> -5/+5V
 $Comp
-L eurogen-rescue:PJ301M-12-eurocad J?
+L eurorack_engine-rescue:PJ301M-12-eurocad-eurogen-rescue J?
 U 1 1 5FB7B91B
 P 10950 7400
 AR Path="/5F91B719/5FB7B91B" Ref="J?"  Part="1"
 AR Path="/5FA42CB5/5FB7B91B" Ref="J9"  Part="1"
+AR Path="/5FB7B91B" Ref="J9"  Part="1"
 F 0 "J9" H 10958 7775 50  0000 C CNN
 F 1 "codec out 4" H 10958 7684 50  0000 C CNN

Commit message: updated schematics
Parts:
- removed J2: cv in 2, Eurocad:PJ301M-12, symbol eurorack_engine-rescue:PJ301M-12-eurocad-eurogen-rescue
- removed J3: cv in 1, Eurocad:PJ301M-12, symbol eurorack_engine-rescue:PJ301M-12-eurocad-eurogen-rescue
- removed J4: codec out 1, Eurocad:PJ301M-12, symbol eurorack_engine-rescue:PJ301M-12-eurocad-eurogen-rescue
- removed J5: codec out 3, Eurocad:PJ301M-12, symbol eurorack_engine-rescue:PJ301M-12-eurocad-eurogen-rescue
- removed J6: cv in 4, Eurocad:PJ301M-12, symbol eurorack_engine-rescue:PJ301M-12-eurocad-eurogen-rescue
- removed J7: cv in 3, Eurocad:PJ301M-12, symbol eurorack_engine-rescue:PJ301M-12-eurocad-eurogen-rescue
- removed J8: codec out 2, Eurocad:PJ301M-12, symbol eurorack_engine-rescue:PJ301M-12-eurocad-eurogen-rescue
- removed J9: codec out 4, Eurocad:PJ301M-12, symbol eurorack_engine-rescue:PJ301M-12-eurocad-eurogen-rescue
- removed R10, R12, R13, R23, R24, R29, R30, R8: 10k, Resistor_THT:R_Axial_DIN0207_L6.3mm_D2.5mm_P7.62mm_Horizontal, symbol Device:R
- removed R11, R14, R25, R26: 200k, Resistor_THT:R_Axial_DIN0207_L6.3mm_D2.5mm_P7.62mm_Horizontal, symbol Device:R
- removed R15, R16, R27, R28: 100k, Resistor_THT:R_Axial_DIN0207_L6.3mm_D2.5mm_P7.62mm_Horizontal, symbol Device:R
- removed R17, R18, R31, R32: 33k, Resistor_THT:R_Axial_DIN0207_L6.3mm_D2.5mm_P7.62mm_Horizontal, symbol Device:R
- removed R19, R20, R21, R22, R33, R34, R7, R9: 1k, Resistor_THT:R_Axial_DIN0207_L6.3mm_D2.5mm_P7.62mm_Horizontal, symbol Device:R
- removed U4: TL074, Package_DIP:DIP-14_W7.62mm_Socket, symbol Amplifier_Operational:TL074
- removed U6: MCP6004, Package_DIP:DIP-14_W7.62mm_Socket, symbol Amplifier_Operational:MCP6004
Other:
- note removed: "CODEC out -> -5/+5V"
- note removed: "CV in -> 0/3V3\n"
- note removed: "INVERTING?"
- note removed: "NON_INVERTING?"
