File: kicad/eurorack_engine/eurorack_engine.kicad_pcb (KiCad board)
At the start: 2 copper layers, 100 x 128 mm, 74 parts, among them IC1 PCM5102, IC2 PCM5102, J1 EURO_PWR_2x5, J2 cv in 2, J3 cv in 1, J4 codec out 1, J5 codec out 3, J6 cv in 4, J7 cv in 3, J8 codec out 2, J9 codec out 4, SW1 SW_Push, SW2 SW_Push, SW3 SW_Push, SW4 SW_Push, U1 ESP32-DEVKITC-32D, U2 LM1117-3.3, U4 TL074, U5 LM4040LP-10, U6 MCP6004, U7 MCP3208

Commit message: schematic update
Parts:
- added SW5: DIP_USBpwr, Button_Switch_THT:SW_DIP_SPSTx01_Slide_9.78x4.72mm_W7.62mm_P2.54mm, F.Cu at (-18.0, 96.5)
- IC1, IC2, U2, U4, U6, U7: moved to F.Cu
- moved U7 237.0 mm to (77.5, 25.0), turned to 90 degrees
- moved U2 222.3 mm to (-3.92, 45.5), turned to 180 degrees
- moved D1 214.4 mm to (24.0, 16.0)
- moved D2 214.4 mm to (37.0, 16.0)
- moved D3 214.4 mm to (50.0, 16.0)
- moved D4 214.4 mm to (63.0, 16.0)
- moved RV1 214.4 mm to (24.0, 73.1)
- moved RV2 214.4 mm to (41.0, 73.4)
- moved RV3 214.4 mm to (58.4, 73.4)
- moved RV4 214.4 mm to (76.0, 73.5)
- moved SW1 214.4 mm to (7.00, 38.0)
- moved SW2 214.4 mm to (69.0, 38.5)
- moved SW3 214.4 mm to (28.0, 38.0)
- moved SW4 214.4 mm to (48.0, 38.5)
- moved U1 214.4 mm to (43.0, 41.0)
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Connections:
- C2 pad 1: +3V3 -> Net-(C2-Pad1)
- C3 pad 2: +3V3 -> Net-(C2-Pad1)
- U2 pad 2: +3V3 -> Net-(C2-Pad1)
Routing:
- added copper zone on F.Cu, net GND
Other:
- board size 100 x 128 mm -> 150.5 x 127 mm

Commit message: updated schematics
Parts:
- removed C8, C9: 100n, Capacitor_THT:C_Disc_D4.3mm_W1.9mm_P5.00mm
- removed SW5: DIP_USBpwr, Button_Switch_THT:SW_DIP_SPSTx01_Slide_9.78x4.72mm_W7.62mm_P2.54mm
- removed U7: MCP3208, Package_DIP:DIP-16_W7.62mm_Socket
- added C4: 100n, Capacitor_THT:C_Disc_D4.3mm_W1.9mm_P5.00mm, F.Cu at (-35.3, -15.4)
- added C5: 100n, Capacitor_THT:C_Disc_D4.3mm_W1.9mm_P5.00mm, F.Cu at (-35.3, -18.9)
- added PWR_SEL1: Conn_01x02, Connector_PinHeader_2.54mm:PinHeader_1x02_P2.54mm_Vertical, F.Cu at (0.96, -63.8)
- added U3: TL074, Package_DIP:DIP-14_W7.62mm_Socket, F.Cu at (-82.5, -64.0)
- J1: value EURO_PWR_2x5 -> cv in 2; footprint Connector_PinHeader_2.54mm:PinHeader_2x05_P2.54mm_Vertical -> Eurocad:PJ301M-12; moved to F.Cu
- J2: value cv in 2 -> cv in 1
- J3: value cv in 1 -> codec out 1
- J4: value codec out 1 -> codec out 3
- J5: value codec out 3 -> cv in 4
- J6: value cv in 4 -> cv in 3
- J7: value cv in 3 -> codec out 2
- J8: value codec out 2 -> codec out 4
- J9: value codec out 4 -> EURO_PWR_2x5; footprint Eurocad:PJ301M-12 -> Connector_PinHeader_2.54mm:PinHeader_2x05_P2.54mm_Vertical
- R10: value 10k -> 200k
- R11: value 200k -> 10k
- R13: value 10k -> 100k
- R14, R25, R26: value 200k -> 100k
- R15, R16: value 100k -> 33k
- R17, R18, R31, R32: value 33k -> 1k
- R21, R22, R9: value 1k -> 200k
- R27, R28: value 100k -> 10k
- R29, R30: value 10k -> 33k
- R33: value 1k -> 4r7
- R34: value 1k -> 2k2
- R5: value 4r7 -> 1k
- R6: value 2k2 -> 1k
- R7: value 1k -> 10k
- U2: value LM1117-3.3 -> MCP3208; footprint Package_TO_SOT_THT:TO-220-3_Vertical -> Package_DIP:DIP-16_W7.62mm
- U4: value TL074 -> MCP6004
- U5: value LM4040LP-10 -> LM1117-3.3; footprint Package_TO_SOT_THT:TO-92_Inline -> Package_TO_SOT_THT:TO-220-3_Vertical
- U6: value MCP6004 -> LM4040LP-10; footprint Package_DIP:DIP-14_W7.62mm_Socket -> Package_TO_SOT_THT:TO-92_Inline
- moved U4 249.6 mm to (-93.3, -42.1)
- moved R7 230.7 mm to (-49.3, -34.8), turned to 0 degrees
- moved C7 229.1 mm to (-70.2, -12.3)
- moved R10 224.8 mm to (-49.3, -30.7)
- moved R13 224.1 mm to (-49.3, -26.7), turned to 0 degrees
- moved R26 209.9 mm to (-56.8, -16.1), turned to 0 degrees
- moved R29 207.6 mm to (-46.0, -18.6), turned to 0 degrees
- moved R9 206.5 mm to (-67.6, -16.1)
- moved R8 206.2 mm to (-67.6, -20.1)
- moved R22 205.2 mm to (-9.94, -51.9), turned to 0 degrees
- moved R33 205.1 mm to (-46.0, -14.5), turned to 0 degrees
- moved R23 204.8 mm to (-46.0, -22.6), turned to 0 degrees
- moved R20 204.4 mm to (-9.94, -47.9), turned to 0 degrees
- moved C6 204.1 mm to (-62.1, -12.3)
- moved R15 202.6 mm to (-78.4, -24.2)
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Connections:
- C6 pad 1: GND -> /aref_-10v
- C6 pad 2: +12V -> GND
- C7 pad 1: -12V -> GND
- C7 pad 2: GND -> +3V3
- IC1 pad 13: (no net) -> /codec_out_1
- IC1 pad 15: (no net) -> /codec_out_2
- IC2 pad 13: (no net) -> /codec_out_3
- IC2 pad 15: (no net) -> /codec_out_4
- J1 pad 1: +12V -> GND
- J1 pad 2: +12V -> (no net)
- J1 pad 3: GND -> Net-(J1-Pad3)
- J9 pad 1: GND -> +12V
- J9 pad 2: (no net) -> +12V
- J9 pad 3: Net-(J9-Pad3) -> GND
- R10 pad 1: Net-(R10-Pad1) -> /aref_-10v
- R10 pad 2: GND -> Net-(R10-Pad2)
- R11 pad 1: /IN_OUT/aref_-10v -> Net-(R11-Pad1)
- R13 pad 1: Net-(R10-Pad1) -> Net-(J1-Pad3)
- R14 pad 1: /IN_OUT/aref_-10v -> Net-(J2-Pad3)
- R14 pad 2: Net-(R14-Pad2) -> Net-(R10-Pad2)
- R15 pad 1: Net-(J2-Pad3) -> Net-(R13-Pad2)
- R15 pad 2: Net-(R11-Pad2) -> /adc_ch1
- R16 pad 1: Net-(J3-Pad3) -> Net-(R10-Pad2)
- R16 pad 2: Net-(R14-Pad2) -> /adc_ch0
- R17 pad 2: /IN_OUT/adc_ch1 -> Net-(J3-Pad3)
- R18 pad 1: Net-(R14-Pad2) -> Net-(R12-Pad2)
- R18 pad 2: /IN_OUT/adc_ch0 -> Net-(J4-Pad3)
- R19 pad 1: Net-(R12-Pad2) -> /codec_out_2
- R19 pad 2: Net-(J4-Pad3) -> Net-(R19-Pad2)
- R20 pad 1: Net-(R13-Pad2) -> /codec_out_4
- R20 pad 2: Net-(J5-Pad3) -> Net-(R20-Pad2)
- R21 pad 1: (no net) -> /aref_-10v
- R22 pad 1: (no net) -> /aref_-10v
- R25 pad 1: /IN_OUT/aref_-10v -> Net-(J5-Pad3)
- R25 pad 2: Net-(R25-Pad2) -> Net-(R21-Pad2)
- R26 pad 1: /IN_OUT/aref_-10v -> Net-(J6-Pad3)
- R26 pad 2: Net-(R26-Pad2) -> Net-(R22-Pad2)
- R27 pad 1: Net-(J6-Pad3) -> Net-(R23-Pad1)
- R27 pad 2: Net-(R25-Pad2) -> Net-(R27-Pad2)
- R28 pad 1: Net-(J7-Pad3) -> Net-(R24-Pad1)
- R28 pad 2: Net-(R26-Pad2) -> Net-(R28-Pad2)
- R29 pad 1: Net-(R23-Pad1) -> Net-(R21-Pad2)
- R29 pad 2: Net-(R29-Pad2) -> /adc_ch3
- R30 pad 1: Net-(R24-Pad1) -> Net-(R22-Pad2)
- R30 pad 2: Net-(R30-Pad2) -> /adc_ch2
- R31 pad 1: Net-(R25-Pad2) -> Net-(R27-Pad2)
- R31 pad 2: /IN_OUT/adc_ch3 -> Net-(J7-Pad3)
- R32 pad 1: Net-(R26-Pad2) -> Net-(R28-Pad2)
- R32 pad 2: /IN_OUT/adc_ch2 -> Net-(J8-Pad3)
- R33 pad 1: Net-(R29-Pad2) -> +12V
- R33 pad 2: Net-(J8-Pad3) -> Net-(C1-Pad1)
- R34 pad 1: Net-(R30-Pad2) -> /aref_-10v
- R34 pad 2: Net-(J9-Pad3) -> -12V
- R5 pad 1: +12V -> /codec_out_1
- R5 pad 2: Net-(C1-Pad1) -> Net-(R5-Pad2)
- R6 pad 1: /POWER/aref_-10v -> /codec_out_3
- R6 pad 2: -12V -> Net-(R6-Pad2)
- R7 pad 1: (no net) -> Net-(R11-Pad1)
- R7 pad 2: Net-(R7-Pad2) -> GND
- R9 pad 1: (no net) -> /aref_-10v
- R9 pad 2: Net-(R9-Pad2) -> Net-(R13-Pad2)
- RV1 pad 2: /ADC/adc_ch4 -> /adc_ch4
- RV2 pad 2: /ADC/adc_ch5 -> /adc_ch6
- RV3 pad 2: /ADC/adc_ch6 -> /adc_ch7
- RV4 pad 2: /ADC/adc_ch7 -> /adc_ch5
- U1 pad 1: (no net) -> +3V3
- U1 pad 10: (no net) -> /adc_cs
- U1 pad 20: (no net) -> GND
- U1 pad 21: (no net) -> /adc_miso
- U1 pad 22: (no net) -> /adc_mosi
- U1 pad 9: (no net) -> /adc_clk
- U2 pad 1: GND -> /adc_ch0
- U2 pad 2: Net-(C2-Pad1) -> /adc_ch1
- U2 pad 3: Net-(C1-Pad1) -> /adc_ch2
- U4 pad 1: Net-(R12-Pad2) -> /adc_ch0
- U4 pad 10: Net-(R7-Pad2) -> GND
- U4 pad 11: -12V -> GND
- U4 pad 12: Net-(R22-Pad2) -> GND
- U4 pad 13: Net-(R24-Pad1) -> Net-(R21-Pad2)
- U4 pad 14: Net-(R30-Pad2) -> /adc_ch3
- U4 pad 2: Net-(R12-Pad1) -> Net-(R10-Pad2)
- U4 pad 3: Net-(R9-Pad2) -> GND
- U4 pad 4: +12V -> +3V3
- U4 pad 5: Net-(R21-Pad2) -> GND
- U4 pad 6: Net-(R23-Pad1) -> Net-(R13-Pad2)
- U4 pad 7: Net-(R29-Pad2) -> /adc_ch1
- U4 pad 8: Net-(R13-Pad2) -> /adc_ch2
- U4 pad 9: Net-(R10-Pad1) -> Net-(R22-Pad2)
- U5 pad 1: (no net) -> GND
- U5 pad 2: GND -> Net-(C2-Pad1)
- U5 pad 3: /POWER/aref_-10v -> Net-(C1-Pad1)
- U6 pad 1: /IN_OUT/adc_ch0 -> (no net)
- U6 pad 2: Net-(R14-Pad2) -> GND
- U6 pad 3: GND -> /aref_-10v
Other:
- board text added: "EURORACK-ENGINE"

Commit message: schematic final
Parts:
- added H1: MountingHole, MountingHole:MountingHole_3.2mm_M3, F.Cu at (15.2, 3.05)
- added H2: MountingHole, MountingHole:MountingHole_3.2mm_M3, F.Cu at (133.6, 3.05)
- added H3: MountingHole, MountingHole:MountingHole_3.2mm_M3, F.Cu at (133.6, 124.0)
- added H4: MountingHole, MountingHole:MountingHole_3.2mm_M3, F.Cu at (15.5, 124.0)
- added H5: MountingHole, MountingHole:MountingHole_3.2mm_M3, F.Cu at (72.6, 3.05)
- added H6: MountingHole, MountingHole:MountingHole_3.2mm_M3, F.Cu at (72.6, 124.0)
- J9: moved to B.Cu
- in 1: renamed from J2
- in 2: renamed from J1
- in 3: renamed from J6
- in 4: renamed from J5
- out 1: renamed from J3
- out 2: renamed from J7
- out 3: renamed from J4
- out 4: renamed from J8
- moved LM1117 241.0 mm to (137.2, 75.4)
- moved R5 232.6 mm to (126.0, 90.9), turned to 270 degrees
- moved MCP6004 228.5 mm to (94.5, 88.1)
- moved J9 228.5 mm to (138.4, 67.3)
- moved MCP3208 223.5 mm to (96.8, 52.8)
- moved R6 211.0 mm to (126.0, 36.3), turned to 270 degrees
- moved C3 208.0 mm to (114.8, 64.8), turned to 90 degrees
- moved R26 206.6 mm to (107.7, 109.0), turned to 180 degrees
- moved R15 205.7 mm to (82.3, 104.1)
- moved R19 205.5 mm to (126.0, 109.7), turned to 90 degrees
- moved R30 205.5 mm to (107.4, 104.1)
- moved C6 203.0 mm to (131.1, 50.3), turned to 270 degrees
- moved TL074 199.9 mm to (98.6, 20.8)
- moved R33 196.1 mm to (130.8, 70.1), turned to 270 degrees
- moved R22 195.4 mm to (115.1, 98.3), turned to 180 degrees
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- renumbered U5 to LM1117, U6 to LM4040, U2 to MCP3208, U4 to MCP6004, IC2 to PCM5102, IC1 to PCM5102, U3 to TL074
Routing:
- net +3V3: track 0.00 -> 359.2 mm
- net /bck2: track 0.00 -> 133.2 mm
- net /lrck2: track 0.00 -> 122.9 mm
- net /din2: track 0.00 -> 119.2 mm
- net /bck1: track 0.00 -> 116.7 mm
- net Net-(J8-Pad3): track 0.00 -> 108.7 mm
- net Net-(R19-Pad2): track 0.00 -> 108.5 mm
- net Net-(J3-Pad3): track 0.00 -> 106.7 mm
- net /aref_-10v: track 0.00 -> 106.7 mm
- net Net-(J4-Pad3): track 0.00 -> 106.1 mm
- net /lrck1: track 0.00 -> 104.7 mm
- net /din1: track 0.00 -> 102.2 mm
- net Net-(R5-Pad2): track 0.00 -> 91.8 mm, vias 0 -> 1
- net /adc_ch4: track 0.00 -> 87.8 mm
- net Net-(J7-Pad3): track 0.00 -> 84.5 mm
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- added copper zone on B.Cu, net GND
Other:
- board text added: "+12V"
- board text added: "-12V"
- board text added: "ENGINE"
- board text added: "EURORACK"
- board text added: "GND"
- board text added: "MUSICAL TECHNOLOGY"
- board text added: "SINNEB"
- board text added: "[¬º-°]¬"
- board text added: "[●▪▪●]"
- board text added: "d[-_-]b"
- board text removed: "EURORACK-ENGINE"
