File: kicad/eurorack_engine/eurorack_engine.sch (KiCad schematic (older format))
At the start: 19 parts, among them IC1 PCM5102, IC2 PCM5102, SW1 SW_Push, SW2 SW_Push, SW3 SW_Push, SW4 SW_Push, U1 ESP32-DEVKITC-32D

Commit message: updated schematics
Parts:
- added C1, C2: 47uf, Capacitor_THT:C_Radial_D6.3mm_H5.0mm_P2.50mm, symbol Device:CP
- added C3, C4, C5, C7: 100n, Capacitor_THT:C_Disc_D4.3mm_W1.9mm_P5.00mm, symbol Device:C
- added C6: 100n, Capacitor_THT:C_Disc_D4.3mm_W1.9mm_P5.00mm, symbol Device:CP
- added J1: cv in 2, Eurocad:PJ301M-12, symbol eurorack_engine-rescue:PJ301M-12-eurocad-eurogen-rescue
- added J2: cv in 1, Eurocad:PJ301M-12, symbol eurorack_engine-rescue:PJ301M-12-eurocad-eurogen-rescue
- added J3: codec out 1, Eurocad:PJ301M-12, symbol eurorack_engine-rescue:PJ301M-12-eurocad-eurogen-rescue
- added J4: codec out 3, Eurocad:PJ301M-12, symbol eurorack_engine-rescue:PJ301M-12-eurocad-eurogen-rescue
- added J5: cv in 4, Eurocad:PJ301M-12, symbol eurorack_engine-rescue:PJ301M-12-eurocad-eurogen-rescue
- added J6: cv in 3, Eurocad:PJ301M-12, symbol eurorack_engine-rescue:PJ301M-12-eurocad-eurogen-rescue
- added J7: codec out 2, Eurocad:PJ301M-12, symbol eurorack_engine-rescue:PJ301M-12-eurocad-eurogen-rescue
- added J8: codec out 4, Eurocad:PJ301M-12, symbol eurorack_engine-rescue:PJ301M-12-eurocad-eurogen-rescue
- added J9: EURO_PWR_2x5, Connector_PinHeader_2.54mm:PinHeader_2x05_P2.54mm_Vertical, symbol eurorack_engine-rescue:EURO_PWR_2x5-eurocad-eurogen-rescue
- added PWR_SEL1: Conn_01x02, Connector_PinHeader_2.54mm:PinHeader_1x02_P2.54mm_Vertical, symbol Connector_Generic:Conn_01x02
- added R10, R21, R22, R9: 200k, Resistor_THT:R_Axial_DIN0207_L6.3mm_D2.5mm_P7.62mm_Horizontal, symbol Device:R
- added R11, R12, R23, R24, R27, R28, R7, R8: 10k, Resistor_THT:R_Axial_DIN0207_L6.3mm_D2.5mm_P7.62mm_Horizontal, symbol Device:R
- added R13, R14, R25, R26: 100k, Resistor_THT:R_Axial_DIN0207_L6.3mm_D2.5mm_P7.62mm_Horizontal, symbol Device:R
- added R15, R16, R29, R30: 33k, Resistor_THT:R_Axial_DIN0207_L6.3mm_D2.5mm_P7.62mm_Horizontal, symbol Device:R
- added R17, R18, R19, R20, R31, R32, R5, R6: 1k, Resistor_THT:R_Axial_DIN0207_L6.3mm_D2.5mm_P7.62mm_Horizontal, symbol Device:R
- added R33: 4r7, Resistor_THT:R_Axial_DIN0207_L6.3mm_D2.5mm_P7.62mm_Horizontal, symbol Device:R
- added R34: 2k2, Resistor_THT:R_Axial_DIN0207_L6.3mm_D2.5mm_P7.62mm_Horizontal, symbol Device:R
- added RV1, RV2, RV3, RV4: R_POT, Potentiometer_THT:Potentiometer_Alps_RK09K_Single_Vertical, symbol Device:R_POT
- added U2: MCP3208, Package_DIP:DIP-16_W7.62mm, symbol Analog_ADC:MCP3208
- added U3: TL074, Package_DIP:DIP-14_W7.62mm_Socket, symbol Amplifier_Operational:TL074
- added U4: MCP6004, Package_DIP:DIP-14_W7.62mm_Socket, symbol Amplifier_Operational:MCP6004
- added U5: LM1117-3.3, Package_TO_SOT_THT:TO-220-3_Vertical, symbol Regulator_Linear:LM1117-3.3
- added U6: LM4040LP-10, Package_TO_SOT_THT:TO-92_Inline, symbol Reference_Voltage:LM4040LP-10
Connections:
- net +3V3: now also U1.1 (3V3), C7.2, PWR_SEL1.1 (Pin_1), RV1.1, RV2.1, RV3.1, RV4.1, U2.15 (Vref), U2.16 (Vdd), U4.4 (V+)
- net GND: now also U1.20 (GND3), C1.2, C2.2, C3.1, C4.1, C5.2, C6.2, C7.1, J1.1, J2.1, J3.1, J4.1, J5.1, J6.1, J7.1, J8.1, J9.3 (GND), J9.4 (GND), J9.5 (GND), J9.6 (GND), J9.7 (GND), J9.8 (GND), R23.2, R24.2, R7.2, R8.2, RV1.3, RV2.3, RV3.3, RV4.3, U2.14 (AGND), U2.9 (DGND), U4.10 (+), U4.11 (V-), U4.12 (+), U4.3 (+), U4.5 (+), U5.1 (GND), U6.2 (K)
- net adc_clk: now also U2.13 (CLK)
- net adc_cs: now also U2.10 (~CS~/SHDN)
- net adc_miso: now also U2.12 (Dout)
- net adc_mosi: now also U2.11 (Din)
- net codec_out_1: now also R5.1
- net codec_out_2: now also R19.1
- net codec_out_3: now also R6.1
- net codec_out_4: now also R20.1
- new net: C2.1, C3.2, PWR_SEL1.2 (Pin_2), U5.2 (VO)
- new net: C1.1, R33.2, U5.3 (VI)
- new net: J1.3, R13.1
- new net: R13.2, R15.1, R9.2, U4.6 (-)
- new net: J6.3, R26.1
- new net: R22.2, R26.2, R30.1, U4.9 (-)
- new net: J5.3, R25.1
- new net: R21.2, R25.2, R29.1, U4.13 (-)
- new net: R11.2, R17.1, U3.1
- new net: R11.1, R7.1, U3.2 (-)
- new net: R5.2, U3.3 (+)
- new net: J3.3, R17.2
- new net: R6.2, U3.10 (+)
- new net: R12.1, R8.1, U3.9 (-)
- new net: R12.2, R18.1, U3.8
- new net: J4.3, R18.2
- new net: R19.2, U3.5 (+)
- new net: R23.1, R27.1, U3.6 (-)
- new net: R27.2, R31.1, U3.7
- new net: J7.3, R31.2
- new net: R20.2, U3.12 (+)
- new net: R24.1, R28.1, U3.13 (-)
- new net: R28.2, R32.1, U3.14
- new net: J8.3, R32.2
- new net: R10.2, R14.2, R16.1, U4.2 (-)
- new net: J2.3, R14.1
- new net +12V: C4.2, J9.1 (+12V), J9.2 (+12V), R33.1, U3.4 (V+)
- new net -12V: C5.1, J9.10 (-12V), J9.9 (-12V), R34.2, U3.11 (V-)
- new net adc_ch0: R16.2, U2.1 (CH0), U4.1
- new net adc_ch1: R15.2, U2.2 (CH1), U4.7
- new net adc_ch2: R30.2, U2.3 (CH2), U4.8
- new net adc_ch3: R29.2, U2.4 (CH3), U4.14
- new net adc_ch4: RV1.2, U2.5 (CH4)
- new net adc_ch5: RV4.2, U2.6 (CH5)
- new net adc_ch6: RV2.2, U2.7 (CH6)
- new net adc_ch7: RV3.2, U2.8 (CH7)
- new net aref_-10v: C6.1, R10.1, R21.1, R22.1, R34.1, R9.1, U6.3 (A)
Other:
- note added: "CODEC out -> -5/+5V"
- note added: "CV in -> 0/3V3\n"
- note added: "INVERTING?"
- note added: "NON_INVERTING?"
- moved on the sheet: IC1, IC2, U1

Commit message: schematic final
Parts:
- added H1, H2, H3, H4, H5, H6: MountingHole, MountingHole:MountingHole_3.2mm_M3, symbol Mechanical:MountingHole
Changed lines of the file:
@@
 Text Label 12200 7900 0    50   ~ 0
 adc_ch0
+$Comp
+L Mechanical:MountingHole H1
+U 1 1 5FA39E89
+P 4950 4850
+F 0 "H1" H 5050 4896 50  0000 L CNN
+F 1 "MountingHole" H 5050 4805 50  0000 L CNN
+F 2 "MountingHole:MountingHole_3.2mm_M3" H 4950 4850 50  0001 C CNN
+F 3 "~" H 4950 4850 50  0001 C CNN
+	1    4950 4850
+	1    0    0    -1
+$EndComp
+$Comp
+L Mechanical:MountingHole H2
+U 1 1 5FA3AFBB
+P 4950 5050
+F 0 "H2" H 5050 5096 50  0000 L CNN
+F 1 "MountingHole" H 5050 5005 50  0000 L CNN
+F 2 "MountingHole:MountingHole_3.2mm_M3" H 4950 5050 50  0001 C CNN
+F 3 "~" H 4950 5050 50  0001 C CNN
+	1    4950 5050
+	1    0    0    -1
+$EndComp
+$Comp
+L Mechanical:MountingHole H3
+U 1 1 5FA3B461
+P 4950 5250
+F 0 "H3" H 5050 5296 50  0000 L CNN
+F 1 "MountingHole" H 5050 5205 50  0000 L CNN
+F 2 "MountingHole:MountingHole_3.2mm_M3" H 4950 5250 50  0001 C CNN
+F 3 "~" H 4950 5250 50  0001 C CNN
+	1    4950 5250
+	1    0    0    -1
+$EndComp
+$Comp
+L Mechanical:MountingHole H4
+U 1 1 5FA3B662
+P 4950 5450
+F 0 "H4" H 5050 5496 50  0000 L CNN
+F 1 "MountingHole" H 5050 5405 50  0000 L CNN
+F 2 "MountingHole:MountingHole_3.2mm_M3" H 4950 5450 50  0001 C CNN
+F 3 "~" H 4950 5450 50  0001 C CNN
+	1    4950 5450
+	1    0    0    -1
+$EndComp
+$Comp
+L Mechanical:MountingHole H5
+U 1 1 5FA3B7D9
+P 4950 5650
+F 0 "H5" H 5050 5696 50  0000 L CNN
+F 1 "MountingHole" H 5050 5605 50  0000 L CNN
+F 2 "MountingHole:MountingHole_3.2mm_M3" H 4950 5650 50  0001 C CNN
+F 3 "~" H 4950 5650 50  0001 C CNN
+	1    4950 5650
+	1    0    0    -1
+$EndComp
+$Comp
+L Mechanical:MountingHole H6
+U 1 1 5FA3B957
+P 4950 5850
+F 0 "H6" H 5050 5896 50  0000 L CNN
+F 1 "MountingHole" H 5050 5805 50  0000 L CNN
+F 2 "MountingHole:MountingHole_3.2mm_M3" H 4950 5850 50  0001 C CNN
+F 3 "~" H 4950 5850 50  0001 C CNN
+	1    4950 5850
+	1    0    0    -1
+$EndComp
 $EndSCHEMATC
